File: pcb/pet_feeder/pet_feeder/pet_feeder.kicad_pcb (KiCad board)
At the start: 2 copper layers, 43.2 x 40.6 mm, 21 parts, among them M0 M0, M1 M1, U1 SiP32431, U2 SiP32431, U3 AP7361C-33E, U4 ESP32-WROOM-32D, U5 INA322

Commit message: Board revision 2 done
Parts:
- renumbered BOOT to BOOT1, RST to RST1
Connections:
- M1 pad 2: /SRV_PWR -> /SRV1_PWR
- RG1 pad 3: Net-(RG1-Pad3) -> /WS_ADC
- U2 pad 1: /WS_3V3 -> /SRV1_PWR
- U2 pad 3: /WS_EN -> /SRV_EN
- U3 pad 1: +BATT -> -BATT
- U3 pad 2: -BATT -> +3V3
- U3 pad 3: +3V3 -> +BATT
- U4 pad 6: Net-(U4-Pad6) -> /WS_ADC
- U5 pad 6: Net-(RG1-Pad3) -> /WS_ADC
Routing:
- net +3V3: track 56.7 -> 118.5 mm
- net /RST: track 0.00 -> 60.4 mm, vias 0 -> 4
- net /WS_ADC: track 0.00 -> 59.1 mm, vias 0 -> 4
- net /~WS_EN: track 0.00 -> 47.8 mm, vias 0 -> 2
- net /REF: track 0.00 -> 22.9 mm
- net /WS_EN: track 18.7 -> 0.00 mm, vias 2 -> 0
- net /SRV1_PWR: track 0.00 -> 14.3 mm
- net /SRV_EN: track 15.0 -> 28.2 mm
- net /WS-: track 0.00 -> 10.5 mm
- net /WS+: track 0.00 -> 8.63 mm
- net /RG: track 0.00 -> 6.49 mm
- net /SRV_PWR: track 19.1 -> 12.9 mm, vias 0 -> 1
- net -BATT: track 50.0 -> 53.9 mm, vias 124 -> 132
- net +BATT: track 65.2 -> 62.4 mm
Other:
- outline, holes or cut-outs redrawn
- board text added: "ESP32 Pet Feeder Module V1.1 Bryan Orabutt 2019"
- board text removed: "ESP32 Pet Feeder Module V1 Bryan Orabutt 2019"
